File: controller/scematic/mqtt-fancontroller-schema.kicad_sch (KiCad schematic)
At the start: 9 parts, among them J1 Fan1, J2 Fan2, J3 Waveshare 1.54inch e-Paper, J4 Barrel_Jack, U1 DS18B20, U2 DS18B20

Commit message: Huge commit, everything is broken now.
Parts:
- removed J2: Fan2, symbol Connector:Conn_01x04_Male
- removed J3: Waveshare 1.54inch e-Paper, symbol Connector:Conn_01x08_Female
- removed U2: DS18B20, Package_TO_SOT_THT:TO-92_Inline, symbol Sensor_Temperature:DS18B20
- added C1, C2, C3, C4, C5: 1 µF, symbol Device:C
- added D2: TX/YELLOW, symbol Device:LED
- added D3: RX/GREEN, symbol Device:LED
- added D4: ALM/RED, symbol Device:LED
- added DS1: HD44780, Display:WC1602A, symbol Display_Character:WC1602A
- added J2: Serial port, symbol Connector:Conn_01x03_Pin
- added R10, R11, R6, R7, R8, R9: 33K, symbol Device:R
- added R12, R13, R14: 1K, symbol Device:R
- added R2: 47, symbol Device:R
- added R3, R4, R5: 1K2, symbol Device:R
- added SW1: SW_SPDT_MSM, symbol Switch:SW_SPDT_MSM
- added SW2, SW3, SW4, SW5: SW_Push, symbol Switch:SW_Push
- added U2: MAX232, symbol Interface_UART:MAX232
- added U3: 74HCT00, symbol 74xx:74HCT00
Connections:
- net +5V: now also C3.2, C4.2, DS1.2 (VDD), R10.1, R2.1, R6.1, R8.1, SW1.1, SW2.2, SW4.2, U2.16 (VCC), U3.14 (VCC)
- net GND: now also C4.1, C5.2, DS1.1 (VSS), DS1.16 (LED(-)), DS1.3 (VO), DS1.5 (R/W), J2.1 (Pin_1), R12.2, R13.2, R14.2, R3.2, R4.1, R5.1, U2.15 (GND), U3.7 (GND)
- net at J1.4 (Pin_4): now also A1.18 (D3); no longer A1.20 (D5)
- net at A1.26 (D11): now also DS1.14 (D7)
- net at A1.28 (D13): now also DS1.6 (E)
- net at A1.25 (D10): now also DS1.13 (D6)
- net at A1.24 (D9): now also DS1.12 (D5)
- net at A1.23 (D8): now also DS1.11 (D4)
- net at A1.22 (D7): now also U2.11 (T1IN), U3.10, U3.9
- net at A1.21 (D6): now also U2.12 (R1OUT), U3.12, U3.13
- net at A1.10 (A1): now also R8.2, R9.1, SW2.1, SW3.2
- net at A1.11 (A2): now also R10.2, R11.1, SW4.1, SW5.2
- net at A1.27 (D12): now also DS1.4 (RS)
- net at A1.9 (A0): now also R6.2, R7.1, SW1.2
- new net: C2.1, U2.4 (C2+)
- new net: C2.2, U2.5 (C2-)
- new net: R13.1, R9.2, SW3.1
- new net: R14.1, R7.2, SW1.3
- new net: C5.1, U2.6 (VS-)
- new net: D3.1 (K), R4.2
- new net: D3.2 (A), U3.11
- new net: DS1.15 (LED(+)), R2.2
- new net: R11.2, R12.1, SW5.1
- new net: D4.1 (K), R5.2
- new net: A1.20 (D5), D4.2 (A)
- new net: C1.1, U2.1 (C1+)
- new net: C1.2, U2.3 (C1-)
- new net: D2.1 (K), R3.1
- new net: D2.2 (A), U3.8
- new net: C3.1, U2.2 (VS+)
- new net: J2.2 (Pin_2), U2.13 (R1IN)
- new net: J2.3 (Pin_3), U2.14 (T1OUT)
Other:
- moved on the sheet: A1, D1, J1, J4, R1, U1
